Commit message: feat: add IMU

File: src/huitzilin_description/urdf/huitzilin.urdf (robot description, URDF)
Before this commit: robot huitzilin, 6 links, 5 joints
Links:
- added link imu_link
Joints:
- added joint base_imu_joint: type fixed, parent base_link, child imu_link, origin xyz=0 0 0 rpy=0 0 0

Commit message: chore: delete rotor links collision blocks and change rotor mass to 0.03

File: src/huitzilin_description/urdf/huitzilin.urdf (robot description, URDF)
Before this commit: robot huitzilin, 7 links, 6 joints
Links:
- link rotor0_link: mass 0.005 -> 0.03; geometry visual mesh filename=package://huitzilin_description/meshes/propeller_ccw.dae scale=0.1 0.1 0.1
- link rotor1_link: mass 0.005 -> 0.03; geometry visual mesh filename=package://huitzilin_description/meshes/propeller_ccw.dae scale=0.1 0.1 0.1
- link rotor2_link: mass 0.005 -> 0.03; geometry visual mesh filename=package://huitzilin_description/meshes/propeller_cw.dae scale=0.1 0.1 0.1
- link rotor3_link: mass 0.005 -> 0.03; geometry visual mesh filename=package://huitzilin_description/meshes/propeller_cw.dae scale=0.1 0.1 0.1
